Commit message: updated

File: src/auv_slam/src/description/orca4_description.urdf (robot description, URDF)
Before this commit: robot orca4_ign, 12 links, 11 joints
Links:
- added link camera_forward_link, mass 0.001; visual box size=0.02 0.02 0.02
Joints:
- added joint camera_forward_joint: type fixed, parent base_link, child camera_forward_link, origin xyz=0.24 0 0 rpy=0 0 0
